File: TempLog.kicad_sch (KiCad schematic)
At the start: 44 parts, among them J1 1.27, 2x5, Male, TH, J3 Conn_01x03, J5 Conn_01x02, J6 USB4105-GF-A-060, J7 Conn_01x02, SW1 SMD_4.6x2.8mm_h1.9mm, SW2 SMD_4.6x2.8mm_h1.9mm, U1 STM32F030C8Tx, U2 GD25Q16CSJGR, U3 TMP1075DGK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

Commit message: Updated BOM. Generated Schematic. Generated Fabrication drawings
Parts:
- C1, C4, C5, C6, C7, C8: Mfg Part# (none) -> GCJ21BR72A104KA01L
- C10, C9: Mfg Part# (none) -> GQM2195C2E200JB12D
- C11, C12: Mfg Part# (none) -> GQM2195C2E4R3BB12D
- C2, C3: value 100nF -> 1uF; Mfg Part# (none) -> GRM21BR71A105KA01L
- D1: Mfg Part# (none) -> 150080VS75000
- D2: Mfg Part# (none) -> 150080RS75000
- J1: Mfg Part# (none) -> HPH2-A-10-UA
- J3: Mfg Part# (none) -> PH1-03-UA
- J5, J7: Mfg Part# (none) -> PH1-02-UA
- J6: Mfg Part# (none) -> USB4105-GF-A-060
- R10, R11: Mfg Part# (none) -> ERJ-6GEYJ101V
- R12, R13, R6: Mfg Part# (none) -> ERJ-6GEYJ103V
- R8: Mfg Part# (none) -> ERJ-6GEYJ511V
- R9: Mfg Part# (none) -> ERJ-6GEYJ331V
- SW1, SW2: Mfg Part# (none) -> KMR441G LFS
- U1: Mfg Part# (none) -> STM32F030C8T6
- U2: Mfg Part# (none) -> GD25Q16ETIGR
- U3: Mfg Part# (none) -> TMP1075DGKR
- U6: Mfg Part# (none) -> MIC5504-3.3YM5-TR
- Y1: value 8.0MHz H130A-8.000-18-2030-EXT-TR -> ABM3-8.000MHZ-J4Q-T; Mfg Part# (none) -> ABM3-8.000MHZ-J4Q-T
- Y2: Mfg Part# (none) -> CC7V-T1A-32.768KHZ-12.5PF-20PPM-TA-QC
